Commit message: Add hokuyo variant

File: urdf/ttb3_hokuyo.urdf.xacro (robot description, xacro)
@@ -133,7 +133,6 @@
   </joint>
   <link name="imu_link"/>
-  <xacro:include filename="$(find turtlebot3_ramp_sim)/urdf/VLP-16.urdf.xacro"/>
-  <VLP-16 parent="base_link" name="velodyne" topic="/velodyne_points" hz="20" min_range="0.1">
-    <origin xyz="-0.05 0 1.0" rpy="0 0 0" />
-  </VLP-16>
+ <!--  Hokuyo Laser Sensor-->
+ <xacro:include filename="$(find turtlebot3_ramp_sim)/urdf/hokuyo.urdf.xacro"/>
+ <sensor_hokuyo parent="base_link"/>
 </robot>
