Commit message: Change IMU

File: urdf/VLP-16.urdf.xacro (robot description, xacro)
@@ -17,5 +17,5 @@
           izz="${0.5 * 0.83 * (0.0516*0.0516)}"/>
       </inertial>
-      -->
+     -->
       <visual>
         <geometry>

File: urdf/ttb3_velodyne.urdf.xacro (robot description, xacro)
@@ -2,5 +2,5 @@
 <robot name="turtlebot3_waffle" xmlns:xacro="http://ros.org/wiki/xacro">
 <xacro:include filename="$(find turtlebot3_description)/urdf/common_properties.xacro"/>
-  <xacro:include filename="$(find turtlebot3_description)/urdf/turtlebot3_waffle.gazebo.xacro"/>
+  <xacro:include filename="$(find turtlebot3_ramp_sim)/urdf/turtlebot3_waffle.gazebo.xacro"/>
   <link name="base_footprint"/>
   <joint name="base_joint" type="fixed">
@@ -135,7 +135,7 @@
   <!-- VLP-16 -->
   <xacro:include filename="$(find turtlebot3_ramp_sim)/urdf/VLP-16.urdf.xacro"/>
-  <VLP-16 parent="base_link" name="velodyne" topic="/velodyne_points" hz="20" min_range="0.1">
+  <VLP-16 parent="base_link" name="velodyne" topic="/velodyne_points" hz="10" min_range="0.1">
 <!--hz="10" samples="360" gpu="false" lasers="16" max_range="100">-->
-    <origin xyz="-0.05 0 1.0" rpy="0 0 0" />
+    <origin xyz="-0 0 1.0" rpy="0 0 0" />
   </VLP-16>
 </robot>
