Commit message: Make changes to URDF and launch file

File: urdf/ttb3_velodyne.urdf.xacro (robot description, xacro)
@@ -130,5 +130,5 @@
     <parent link="base_link"/>
     <child link="imu_link"/>
-    <origin xyz="0.0 0 0.068" rpy="0 0 0"/>
+    <origin xyz="0.0 0 1.0" rpy="0 0 0"/> <!-- z = 0.068 -->
   </joint>
   <link name="imu_link"/>
@@ -137,5 +137,5 @@
   <VLP-16 parent="base_link" name="velodyne" topic="/velodyne_points" hz="10" min_range="0.1">
 <!--hz="10" samples="360" gpu="false" lasers="16" max_range="100">-->
-    <origin xyz="-0 0 1.0" rpy="0 0 0" />
+    <origin xyz="0 0 1.0" rpy="0 0 0" />
   </VLP-16>
 </robot>

File: urdf/turtlebot3_waffle.gazebo.xacro (robot description, xacro)
@@ -77,12 +77,12 @@
     <plugin name="imu_plugin" filename="libhector_gazebo_ros_imu.so">
       <robotNamespace>/</robotNamespace>
-      <updateRate>50.0</updateRate>
+      <updateRate>10.0</updateRate> <!-- 50.0 -->
       <bodyName>imu_link</bodyName>
       <topicName>imu/data</topicName>
-      <accelDrift>0.005 0.005 0.005</accelDrift>
+      <accelDrift>0.005 0.005 0.005</accelDrift> <!-- 0.005 0.005 0.005 -->
       <accelGaussianNoise>0.005 0.005 0.005</accelGaussianNoise>
-      <rateDrift>0.005 0.005 0.005 </rateDrift>
+      <rateDrift>0.005 0.005 0.005</rateDrift>
       <rateGaussianNoise>0.005 0.005 0.005 </rateGaussianNoise>
-      <headingDrift>0.005</headingDrift>
+      <headingDrift>0.005</headingDrift> <!-- 0.005 -->
       <headingGaussianNoise>0.005</headingGaussianNoise>
     </plugin>
@@ -118,78 +118,3 @@
   </gazebo>
 -->
-  <gazebo reference="base_scan">
-    <material>Gazebo/FlatBlack</material>
-    <sensor type="ray" name="lds_lfcd_sensor">
-      <pose>0 0 0 0 0 0</pose>
-      <visualize>$(arg laser_visual)</visualize>
-      <update_rate>5</update_rate>
-      <ray>
-        <scan>
-          <horizontal>
-            <samples>360</samples>
-            <resolution>1</resolution>
-            <min_angle>0.0</min_angle>
-            <max_angle>6.28319</max_angle>
-          </horizontal>
-        </scan>
-        <range>
-          <min>0.120</min>
-          <max>3.5</max>
-          <resolution>0.015</resolution>
-        </range>
-        <noise>
-          <type>gaussian</type>
-          <mean>0.0</mean>
-          <stddev>0.01</stddev>
-        </noise>
-      </ray>
-      <plugin name="gazebo_ros_lds_lfcd_controller" filename="libgazebo_ros_laser.so">
-        <topicName>scan</topicName>
-        <frameName>base_scan</frameName>
-      </plugin>
-    </sensor>
-  </gazebo>
-  <gazebo reference="camera_rgb_frame">
-    <sensor type="depth" name="realsense_R200">
-      <always_on>true</always_on>
-      <visualize>$(arg camera_visual)</visualize>
-      <camera>
-          <horizontal_fov>1.3439</horizontal_fov>
-          <image>
-              <width>1920</width>
-              <height>1080</height>
-              <format>R8G8B8</format>
-          </image>
-          <depth_camera></depth_camera>
-          <clip>
-              <near>0.03</near>
-              <far>100</far>
-          </clip>
-      </camera>
-      <plugin name="camera_controller" filename="libgazebo_ros_openni_kinect.so">
-        <baseline>0.2</baseline>
-        <alwaysOn>true</alwaysOn>
-        <updateRate>30.0</updateRate>
-        <cameraName>camera</cameraName>
-        <frameName>camera_rgb_optical_frame</frameName>
-        <imageTopicName>rgb/image_raw</imageTopicName>
-        <depthImageTopicName>depth/image_raw</depthImageTopicName>
-        <pointCloudTopicName>depth/points</pointCloudTopicName>
-        <cameraInfoTopicName>rgb/camera_info</cameraInfoTopicName>
-        <depthImageCameraInfoTopicName>depth/camera_info</depthImageCameraInfoTopicName>
-        <pointCloudCutoff>0.4</pointCloudCutoff>
-            <hackBaseline>0.07</hackBaseline>
-            <distortionK1>0.0</distortionK1>
-            <distortionK2>0.0</distortionK2>
-            <distortionK3>0.0</distortionK3>
-            <distortionT1>0.0</distortionT1>
-            <distortionT2>0.0</distortionT2>
-        <CxPrime>0.0</CxPrime>
-        <Cx>0.0</Cx>
-        <Cy>0.0</Cy>
-        <focalLength>0</focalLength>
-        <hackBaseline>0</hackBaseline>
-      </plugin>
-    </sensor>
-  </gazebo>
 </robot>

Commit message: Change IMU update rate to 10hz

File: urdf/ttb3_velodyne.urdf.xacro (robot description, xacro)
@@ -130,5 +130,5 @@
     <parent link="base_link"/>
     <child link="imu_link"/>
-    <origin xyz="0.0 0 1.0" rpy="0 0 0"/> <!-- z = 0.068 -->
+    <origin xyz="0.0 0 0.068" rpy="0 0 0"/> <!-- z = 0.068 -->
   </joint>
   <link name="imu_link"/>

File: urdf/turtlebot3_waffle.gazebo.xacro (robot description, xacro)
@@ -77,5 +77,5 @@
     <plugin name="imu_plugin" filename="libhector_gazebo_ros_imu.so">
       <robotNamespace>/</robotNamespace>
-      <updateRate>500.0</updateRate>
+      <updateRate>10.0</updateRate>
       <bodyName>imu_link</bodyName>
       <frameName>imu_link</frameName>
